File: fsrKeyer.kicad_sch (KiCad schematic)
At the start: 24 parts, among them J1 PJ-313, Q1 2N7000, Q11 SI2300, Q12 SI2300, Q2 2N7000

Commit message: Accommodate smaller and/or shorter and/or longer sensors. Gerbers sent to DKRed for fabrication.
Parts:
- S1, S2: footprint ac8es:FSR_RP-C18.3-ST_SMD -> ac8es:FSR_RP-C18.3-ST_RP-C10ST_SMD; Alt1Datasheet (none) -> https://www.alibaba.com/product-detail/FSR-Single-Zone-Sens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; Alt1PartNum (none) -> RP-C10-ST; Alt2Datasheet (none) -> https://www.alibaba.com/product-detail/Single-Zone-0-40mm-T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; Alt2PartNum (none) -> RP-C10-LT
Changed lines of the file:
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@@
 	(title_block
 		(title "Paddle Keyer")
-		(date "2025-10-31")
-		(rev "0.1")
+		(date "2026-04-23")
+		(rev "0.2")
 		(comment 1 "Artwork (C)2025 AC8ES")
 		(comment 2 "and mods by UD6ARJ, https://telegra.ph/CW-key-05-25")
@@
 			)
 		)
-		(property "Footprint" "ac8es:FSR_RP-C18.3-ST_SMD"
+		(property "Footprint" "ac8es:FSR_RP-C18.3-ST_RP-C10ST_SMD"
 			(at 115.062 71.12 90)
 			(effects
@@
 			)
 		)
-		(property "Datasheet" "~"
+		(property "Datasheet" "https://www.alibaba.com/product-detail/Intelligent-FSR-402-Thin-Film-Pressure_1600649457578.html"
 			(at 116.84 71.12 0)
 			(effects
@@
 			)
 		)
+		(property "Alt1Datasheet" "https://www.alibaba.com/product-detail/FSR-Single-Zone-Sensor-RP-C10_1600972475459.html"
+			(at 116.84 71.12 0)
+			(effects
+				(font
+					(size 1.27 1.27)
+				)
+				(hide yes)
+			)
+		)
+		(property "Alt1PartNum" "RP-C10-ST"
+			(at 116.84 71.12 0)
+			(effects
+				(font
+					(size 1.27 1.27)
+				)
+				(hide yes)
+			)
+		)
+		(property "Alt2Datasheet" "https://www.alibaba.com/product-detail/Single-Zone-0-40mm-Thin-Film_1600949339963.html"
+			(at 116.84 71.12 0)
+			(effects
+				(font
+					(size 1.27 1.27)
+				)
+				(hide yes)
+			)
+		)
+		(property "Alt2PartNum" "RP-C10-LT"
+			(at 116.84 71.12 0)
+			(effects
+				(font
+					(size 1.27 1.27)
+				)
+				(hide yes)
+			)
+		)
 		(pin "1"
 		)
@@
 		(on_board yes)
 		(dnp no)
-		(fields_autoplaced yes)
 		(property "Reference" "S1"
 			(at 120.65 40.6018 0)
@@
 			)
 		)
-		(property "Footprint" "ac8es:FSR_RP-C18.3-ST_SMD"
+		(property "Footprint" "ac8es:FSR_RP-C18.3-ST_RP-C10ST_SMD"
 			(at 115.062 41.91 90)
 			(effects
@@
 			)
 		)
-		(property "Datasheet" "~"
+		(property "Datasheet" "https://www.alibaba.com/product-detail/Intelligent-FSR-402-Thin-Film-Pressure_1600649457578.html"
 			(at 116.84 41.91 0)
 			(effects
@@
 			(at 116.84 41.91 0)
 			(effects
+				(font
+					(size 1.27 1.27)
+				)
+				(hide yes)
+			)
+		)
+		(property "Alt1PartNum" "RP-C10-ST"
+			(at 126.746 44.958 0)
+			(effects
+				(font
+					(size 1.27 1.27)
+				)
+				(hide yes)
+			)
+		)
+		(property "Alt1Datasheet" "https://www.alibaba.com/product-detail/FSR-Single-Zone-Sensor-RP-C10_1600972475459.html"
+			(at 116.84 41.91 0)
+			(effects
+				(font
+					(size 1.27 1.27)
+				)
+				(hide yes)
+			)
+		)
+		(property "Alt2PartNum" "RP-C10-LT"
+			(at 126.746 46.482 0)
+			(effects
+				(font
+					(size 1.27 1.27)
+				)
+				(hide yes)
+			)
+		)
+		(property "Alt2Datasheet" "https://www.alibaba.com/product-detail/Single-Zone-0-40mm-Thin-Film_1600949339963.html"
+			(at 116.84 41.91 0)
+			(effects
