File: fsrKeyer.kicad_pcb (KiCad board)
At the start: 2 copper layers, 47.9 x 19.2 mm, 23 parts, among them J1 AudioJack3, Q1 2N7000, Q11 2N7002, Q12 2N7002, Q2 2N7000

Commit message: Check in v0.2 of fsrKeyer.kicad_pcb.
Parts:
- Q11, Q12: value 2N7002 -> SI2300
- S1, S2: footprint ac8es:FSR_RP-C18.3-ST_SMD -> ac8es:FSR_RP-C18.3-ST_RP-C10ST_SMD
Routing:
- net /Ring: track 35.5 -> 51.3 mm
- net /Tip: track 34.4 -> 41.2 mm, vias 3 -> 2
- net GND: vias 76 -> 72
Other:
- board size 47.9 x 19.2 mm -> 47.8 x 19.2 mm
- board text added: "${COMMENT1} ${COMMENT2} ${COMMENT3} ${COMMENT4} ${COMMENT5} ${COMMENT6}; v${REVISION}"
- board text added: "${COMMENT7}"
- board text removed: "${COMMENT1} ${COMMENT2} ${COMMENT3} ${COMMENT4} Artwork (C)2025 AC8ES; v${REVISION}"
